File: kicad/air_sensor/mics6814.kicad_sch (KiCad schematic)
At the start: 23 parts, among them M1 MiCS-6814, U6 ATtiny214

Commit message: updated schema
added 5V 3A buck converter
refined 3v3 LDO
added symbols for new components
added text comments for designing the pcb
Parts:
- removed C12: 4.7uF, symbol Device:C
- removed C13, C16: 103, symbol Device:C
- removed C14: 104, symbol Device:C
- removed C15: 106, symbol Device:C
- removed C18: 100nF, symbol Device:C
- removed R1, R4: 100R, symbol Device:R
- removed R19, R20: 4.7K, symbol Device:R
- removed R2, R3: 10K, symbol Device:R
- removed R5: 400K, symbol Device:R
- removed U6: ATtiny214, symbol air_sens_lib:ATtiny214
- added C12: 4.7uF, symbol common:Capacitor
- added C13, C14, C15: 103, symbol common:Capacitor
- added C16: 106, symbol common:Capacitor
- added C18, C23: 100nF, symbol common:Capacitor
- added J1: Program Header, symbol air_sens_lib:ATtiny1614_programming_header
- added R1, R4: 100R, symbol common:Resistor
- added R2, R3: 10K, symbol common:Resistor
- added R5: 400K, symbol common:Resistor
- added U6: ~, symbol air_sens_lib:ATtiny1614
- added U9: Buffer, symbol air_sens_lib:SN74LVC125
- A1: value AD8552M -> AD8552
Connections:
- net +5V: no longer G2.2 (Vin), R10.2, R11.2, R12.1
- net CO_VAL: now also U6.3 (PA5)
- net GND: now also C12.2, C13.1, C14.1, C16.1, J1.2 (GND), R1.2, R3.1, U6.14 (GND), U9.1 (1OE), U9.4 (2OE), U9.7 (GND); no longer A1.7 (INB-), A1.8 (INB+)
- net NH3_VAL: now also U6.4 (PA6)
- net NO2_VAL: now also U6.5 (PA7)
- net SCL: now also U6.9 (PB0)
- net SDA: now also U6.8 (PB1)
- net at O1.1 (Vsensor+): now also C12.1, R1.1, R2.1
- net at A1.3 (+IN_A): now also R2.2
- net at A1.2 (-IN_A): now also C15.2, R3.2, R5.2
- net at A1.1 (OUT_A): now also C15.1, R4.2, R5.1
- net +3.3V: no longer names the net of A1.5 (+IN_B)
- net +3.3V: no longer G2.1 (VCC)
- net RX renamed C02_RX
- net C02_RX: now also U9.6 (2Y)
- net TX renamed CO2_TX
- net CO2_TX: now also U9.2 (1A)
- new net: C23.1, U9.14 (VCC)
- new net: C18.2, U6.1 (VDD)
- new net 02_A: C16.2, R4.1, U6.2 (PA4)
- new net 3V3: A1.8 (+Vs), C13.2, C14.2, C18.1, C23.2, G2.1 (3V3), J1.1 (VCC)
- new net 5V: G2.2 (5V), R10.2, R11.2, R12.1
- new net AT_RX: U6.12 (PA2), U9.3 (1Y)
- new net AT_TX: U6.11 (PA1), U9.5 (2A)
- new net UPDI: J1.3 (UPDI), U6.10 (PA0/RST/UPDI)
- no-connect marks 7 -> 14

Commit message: updated power symbol labels, replaced power symbols in schematic with our own custom symbols
Connections:
- net +5V is gone; now on net 5V: C32.2
- net AT_RX renamed AT_GAS_RX
- net AT_TX renamed AT_GAS_TX
