File: hardware/boards/vehicle/car/car.kicad_sch (KiCad schematic)
At the start: 23 parts, among them J1 Conn_01x04_Socket, J2 Conn_01x05_Socket, J3 Conn_01x05_Socket, J4 Conn_01x05_Socket, J5 Conn_01x02_Socket, SW1 SW_SPST, SW2 SW_Push, U1 ATmega328P-A, Y1 16MHz

Commit message: car schematic
Changed lines of the file:
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@@
 	)
 	(junction
+		(at 233.68 36.83)
+		(diameter 0)
+		(color 0 0 0 0)
+	)
+	(junction
 		(at 226.06 39.37)
 		(diameter 0)
@@
 	(wire
 		(pts
+			(xy 226.06 36.83) (xy 233.68 36.83)
+		)
+		(stroke
+			(width 0)
+			(type default)
+		)
+	)
+	(wire
+		(pts
 			(xy 241.3 128.27) (xy 243.84 128.27)
 		)
@@
 	(wire
 		(pts
-			(xy 226.06 36.83) (xy 233.68 36.83)
+			(xy 93.98 120.65) (xy 95.25 120.65)
 		)
 		(stroke
@@
 	(wire
 		(pts
-			(xy 93.98 120.65) (xy 95.25 120.65)
+			(xy 67.31 30.48) (xy 67.31 31.75)
 		)
 		(stroke
@@
 	(wire
 		(pts
-			(xy 67.31 30.48) (xy 67.31 31.75)
+			(xy 110.49 115.57) (xy 110.49 120.65)
 		)
 		(stroke
@@
 	(wire
 		(pts
-			(xy 110.49 115.57) (xy 110.49 120.65)
+			(xy 233.68 36.83) (xy 242.57 36.83)
 		)
 		(stroke
@@
 		)
 	)
+	(wire
+		(pts
+			(xy 242.57 26.67) (xy 242.57 36.83)
+		)
+		(stroke
+			(width 0)
+			(type default)
+		)
+	)
 	(global_label "M1_PWM_CW"
 		(shape input)
@@
 					(unit 1)
 				)
+			)
+		)
+	)
+	(symbol
+		(lib_id "power:PWR_FLAG")
+		(at 242.57 26.67 0)
+		(unit 1)
+		(exclude_from_sim no)
+		(in_bom yes)
+		(on_board yes)
+		(dnp no)
+		(fields_autoplaced yes)
+		(property "Reference" "#FLG03"
+			(at 242.57 24.765 0)
+			(effects
+				(font
+					(size 1.27 1.27)
+				)
+				(hide yes)
+			)
+		)
+		(property "Value" "PWR_FLAG"
+			(at 242.57 21.59 0)
+			(effects
+				(font
+					(size 1.27 1.27)
+				)
+			)
+		)
+		(property "Footprint" ""
+			(at 242.57 26.67 0)
+			(effects
+				(font
+					(size 1.27 1.27)
+				)
+				(hide yes)
+			)
+		)
+		(property "Datasheet" "~"
+			(at 242.57 26.67 0)
+			(effects
+				(font
+					(size 1.27 1.27)
+				)
+				(hide yes)
+			)
+		)
+		(property "Description" "Special symbol for telling ERC where power comes from"
+			(at 242.57 26.67 0)
+			(effects
+				(font
+					(size 1.27 1.27)
+				)
+				(hide yes)
+			)
+		)
+		(pin "1"
+		)
+		(instances
+			(project ""
+				(path "/d4bcaa97-404f-4040-88d9-84162ce8c00c"
+					(reference "#FLG03")
+					(unit 1)
+				)
