File: hardware/boards/vehicle/car/car.kicad_sch (KiCad schematic)
At the start: 23 parts, among them J1 Conn_01x04_Socket, J2 Conn_01x05_Socket, J3 Conn_01x05_Socket, J4 Conn_01x05_Socket, J5 Conn_01x02_Socket, SW1 SW_SPST, SW2 SW_Push, U1 ATmega328P-A, Y1 8MHz

Commit message: pcb for car
Parts:
- removed SW1: SW_SPST, Connector_PinHeader_2.54mm:PinHeader_1x02_P2.54mm_Vertical, symbol Switch:SW_SPST
- renumbered SW2 to SW1
Connections:
- net Power/VIN: now also BT1.1 (+)
Other:
- moved on the sheet: D1, R1
