File: hardware/boards/vehicle/car/car.kicad_pcb (KiCad board)
At the start: 2 copper layers, 0 parts

Commit message: corrected SD card and transceiver on symbol and schema
Parts:
- added BT1: Battery 12V, Connector_PinHeader_2.54mm:PinHeader_1x02_P2.54mm_Vertical, F.Cu at (146.8, 107.3)
- added C1: 100nF, Capacitor_SMD:C_0603_1608Metric_Pad1.08x0.95mm_HandSolder, F.Cu at (142.3, 91.5)
- added C13: 470uF, Capacitor_THT:CP_Radial_D10.0mm_P5.00mm, F.Cu at (263.3, 26.0)
- added C14: 100nF, Capacitor_SMD:C_0603_1608Metric_Pad1.08x0.95mm_HandSolder, F.Cu at (250.4, 45.3)
- added C15: 470uF, Capacitor_THT:CP_Radial_D10.0mm_P5.00mm, F.Cu at (263.3, 37.5)
- added C16: 100nF, Capacitor_SMD:C_0603_1608Metric_Pad1.08x0.95mm_HandSolder, F.Cu at (250.4, 47.8)
- added C19: 10uF, Capacitor_THT:CP_Radial_D5.0mm_P2.00mm, F.Cu at (21.6, 23.7)
- added C2: 12pF, Capacitor_SMD:C_0603_1608Metric_Pad1.08x0.95mm_HandSolder, F.Cu at (142.3, 94.0)
- added C20: 100nF, Capacitor_SMD:C_0603_1608Metric_Pad1.08x0.95mm_HandSolder, F.Cu at (28.1, 21.7)
- added C21: 100nF, Capacitor_SMD:C_0603_1608Metric_Pad1.08x0.95mm_HandSolder, F.Cu at (28.1, 24.2)
- added C22: 22uF, Capacitor_SMD:C_0603_1608Metric_Pad1.08x0.95mm_HandSolder, F.Cu at (28.1, 26.7)
- added C23: 22uF, Capacitor_SMD:C_0603_1608Metric_Pad1.08x0.95mm_HandSolder, F.Cu at (28.1, 29.2)
- added C24: 75pF, Capacitor_SMD:C_0603_1608Metric_Pad1.08x0.95mm_HandSolder, F.Cu at (32.4, 21.7)
- added C25: 10nF, common:C_0603, F.Cu at (22.9, 165.7)
- added C26: 1nF, common:C_0603, F.Cu at (22.9, 168.2)
- added C27: 33nF, common:C_0603, F.Cu at (22.9, 170.8)
- added C28: 12pF, common:C_0603, F.Cu at (22.9, 173.3)
- added C29: 12pF, common:C_0603, F.Cu at (22.9, 175.8)
- added C3: 12pF, Capacitor_SMD:C_0603_1608Metric_Pad1.08x0.95mm_HandSolder, F.Cu at (142.3, 96.6)
- added C30: 2.2nF, common:C_0603, F.Cu at (22.9, 178.4)
- added C31: 4.7nF, common:C_0603, F.Cu at (22.9, 180.9)
- added C32: 1.5pF, common:C_0603, F.Cu at (27.0, 165.7)
- added C33: 1.0pF, common:C_0603, F.Cu at (27.0, 168.2)
- added C34: 220pF, common:C_0603, F.Cu at (27.0, 170.8)
- added C35: 1uF, common:C_0603, F.Cu at (27.0, 173.3)
- added C36: 0.3pF, common:C_0603, F.Cu at (27.0, 175.8)
- added C37: 1.5pF, common:C_0603, F.Cu at (27.0, 178.4)
- added C38: 1.5pF, common:C_0603, F.Cu at (27.0, 180.9)
- added C39: 1.5pF, common:C_0603, F.Cu at (31.1, 165.7)
- added C4: 100nF, Capacitor_SMD:C_0603_1608Metric_Pad1.08x0.95mm_HandSolder, F.Cu at (142.3, 99.1)
- added C40: 1.5pF, common:C_0603, F.Cu at (31.1, 168.2)
- added C41: 22uF, Capacitor_THT:CP_Radial_D5.0mm_P2.00mm, F.Cu at (21.6, 30.3)
- added C42: 100nF, Capacitor_SMD:C_0603_1608Metric_Pad1.08x0.95mm_HandSolder, F.Cu at (32.4, 24.2)
- added C43: 22uF, Capacitor_THT:CP_Radial_D5.0mm_P2.00mm, F.Cu at (21.6, 36.8)
- added C5: 10uF, Capacitor_SMD:C_0603_1608Metric_Pad1.08x0.95mm_HandSolder, F.Cu at (268.5, 143.4)
- added C6: 100nF, Capacitor_SMD:C_0603_1608Metric_Pad1.08x0.95mm_HandSolder, F.Cu at (268.5, 145.9)
- added D1: LED, LED_SMD:LED_0603_1608Metric_Pad1.05x0.95mm_HandSolder, F.Cu at (165.1, 91.6)
- added D10: UF5408, Diode_THT:D_DO-201AD_P15.24mm_Horizontal, F.Cu at (230.6, 64.1)
- added D11: UF5408, Diode_THT:D_DO-201AD_P15.24mm_Horizontal, F.Cu at (230.6, 70.8)
- added D12: 1N400x, Diode_THT:D_DO-41_SOD81_P2.54mm_Vertical_AnodeUp, F.Cu at (39.8, 41.1)
- added D2: LED, LED_SMD:LED_0603_1608Metric_Pad1.05x0.95mm_HandSolder, F.Cu at (165.1, 94.2)
- added D3: LED, LED_SMD:LED_0603_1608Metric_Pad1.05x0.95mm_HandSolder, F.Cu at (165.1, 96.8)
- added D4: UF5408, Diode_THT:D_DO-201AD_P15.24mm_Horizontal, F.Cu at (230.6, 23.6)
- added D5: UF5408, Diode_THT:D_DO-201AD_P15.24mm_Horizontal, F.Cu at (230.6, 30.4)
- added D6: UF5408, Diode_THT:D_DO-201AD_P15.24mm_Horizontal, F.Cu at (230.6, 37.1)
- added D7: UF5408, Diode_THT:D_DO-201AD_P15.24mm_Horizontal, F.Cu at (230.6, 43.9)
- added D8: UF5408, Diode_THT:D_DO-201AD_P15.24mm_Horizontal, F.Cu at (230.6, 50.6)
- added D9: UF5408, Diode_THT:D_DO-201AD_P15.24mm_Horizontal, F.Cu at (230.6, 57.4)
- added J1: Conn_01x04_Socket, Connector_PinHeader_2.54mm:PinHeader_1x04_P2.54mm_Vertical, F.Cu at (160.6, 92.6)
- added J10: Conn_02x03_Odd_Even, Connector_PinHeader_2.54mm:PinHeader_2x03_P2.54mm_Vertical, F.Cu at (268.6, 134.8)
- added J2: Conn_01x05_Socket, Connector_PinHeader_2.54mm:PinHeader_1x05_P2.54mm_Vertical, F.Cu at (146.8, 92.6)
- added J3: Conn_01x05_Socket, Connector_PinHeader_2.54mm:PinHeader_1x05_P2.54mm_Vertical, F.Cu at (151.4, 92.6)
- added J4: Conn_01x05_Socket, Connector_PinHeader_2.54mm:PinHeader_1x05_P2.54mm_Vertical, F.Cu at (156.0, 92.6)
- added J5: Conn_01x02_Socket, Connector_PinHeader_2.54mm:PinHeader_1x02_P2.54mm_Vertical, F.Cu at (151.4, 107.3)
- added J6: SMA, connector:SMA, F.Cu at (42.1, 181.2)
- added J7: 02x04, connector:Pin_02x04, F.Cu at (39.6, 166.6)
- added J8: Conn_01x04_Socket, Connector_PinHeader_2.54mm:PinHeader_1x04_P2.54mm_Vertical, F.Cu at (28.2, 32.8)
- added J9: Conn_02x05_Odd_Even, Connector_PinHeader_2.54mm:PinHeader_2x05_P2.54mm_Vertical, F.Cu at (270.1, 46.3)
- added L1: 10uH, Inductor_SMD:L_0603_1608Metric_Pad1.05x0.95mm_HandSolder, F.Cu at (32.4, 26.7)
- added L10: 2.4nH, common:L_0603, F.Cu at (31.1, 180.9)
- added L6: 8.2nH, common:L_0603, F.Cu at (31.1, 170.8)
- added L7: 2.7nH, common:L_0603, F.Cu at (31.1, 173.3)
- added L8: 3.9nH, common:L_0603, F.Cu at (31.1, 175.8)
- added L9: 2.4nH, common:L_0603, F.Cu at (31.1, 178.4)
- added M1: Motor_DC, Connector_PinHeader_2.54mm:PinHeader_1x02_P2.54mm_Vertical, F.Cu at (250.5, 63.9)
- added M2: Motor_DC, Connector_PinHeader_2.54mm:PinHeader_1x02_P2.54mm_Vertical, F.Cu at (255.1, 63.9)
- added Q1: FQP27P06, Package_TO_SOT_THT:TO-220-3_Vertical, F.Cu at (251.4, 24.1)
- added Q10: AO3400A, Package_TO_SOT_SMD:SOT-23, F.Cu at (274.0, 35.8)
- added Q11: 2N3904, Package_TO_SOT_THT:TO-92_Inline, F.Cu at (263.2, 58.9)
- added Q12: 2N3904, Package_TO_SOT_THT:TO-92_Inline, F.Cu at (263.2, 64.7)
- added Q2: AO3400A, Package_TO_SOT_SMD:SOT-23, F.Cu at (274.0, 22.4)
- added Q3: FQP27P06, Package_TO_SOT_THT:TO-220-3_Vertical, F.Cu at (251.4, 30.1)
- added Q4: AO3400A, Package_TO_SOT_SMD:SOT-23, F.Cu at (274.0, 26.9)
- added Q5: 2N3904, Package_TO_SOT_THT:TO-92_Inline, F.Cu at (263.2, 47.3)
- added Q6: 2N3904, Package_TO_SOT_THT:TO-92_Inline, F.Cu at (263.2, 53.1)
- added Q7: FQP27P06, Package_TO_SOT_THT:TO-220-3_Vertical, F.Cu at (251.4, 36.0)
- added Q8: AO3400A, Package_TO_SOT_SMD:SOT-23, F.Cu at (274.0, 31.4)
- added Q9: FQP27P06, Package_TO_SOT_THT:TO-220-3_Vertical, F.Cu at (251.4, 42.0)
- added R1: 680, Resistor_SMD:R_0603_1608Metric_Pad0.98x0.95mm_HandSolder, F.Cu at (142.3, 101.6)
- added R10: 10K, Resistor_SMD:R_0603_1608Metric_Pad0.98x0.95mm_HandSolder, F.Cu at (250.4, 57.8)
- added R11: 10K, Resistor_SMD:R_0603_1608Metric_Pad0.98x0.95mm_HandSolder, F.Cu at (250.4, 60.3)
- added R12: 4.7K, Resistor_SMD:R_0603_1608Metric_Pad0.98x0.95mm_HandSolder, F.Cu at (254.7, 45.3)
- added R13: 47, Resistor_SMD:R_0603_1608Metric_Pad0.98x0.95mm_HandSolder, F.Cu at (254.7, 47.8)
- added R14: 1K, Resistor_SMD:R_0603_1608Metric_Pad0.98x0.95mm_HandSolder, F.Cu at (254.7, 50.3)
- added R15: 1K, Resistor_SMD:R_0603_1608Metric_Pad0.98x0.95mm_HandSolder, F.Cu at (254.7, 52.8)
- added R16: 47, Resistor_SMD:R_0603_1608Metric_Pad0.98x0.95mm_HandSolder, F.Cu at (254.7, 55.3)
- added R17: 4.7K, Resistor_SMD:R_0603_1608Metric_Pad0.98x0.95mm_HandSolder, F.Cu at (254.7, 57.8)
- added R18: 10K, Resistor_SMD:R_0603_1608Metric_Pad0.98x0.95mm_HandSolder, F.Cu at (254.7, 60.3)
- added R19: 10K, Resistor_SMD:R_0603_1608Metric_Pad0.98x0.95mm_HandSolder, F.Cu at (259.1, 45.3)
- added R2: 10K, Resistor_SMD:R_0603_1608Metric_Pad0.98x0.95mm_HandSolder, F.Cu at (142.3, 104.1)
- added R20: 4.7K, Resistor_SMD:R_0603_1608Metric_Pad0.98x0.95mm_HandSolder, F.Cu at (259.1, 47.8)
- added R21: 47, Resistor_SMD:R_0603_1608Metric_Pad0.98x0.95mm_HandSolder, F.Cu at (259.1, 50.3)
- added R22: 1K, Resistor_SMD:R_0603_1608Metric_Pad0.98x0.95mm_HandSolder, F.Cu at (259.1, 52.8)
- added R23: 511K, Resistor_SMD:R_0603_1608Metric_Pad0.98x0.95mm_HandSolder, F.Cu at (32.4, 29.2)
- added R24: 22k, common:R_0603, F.Cu at (35.3, 165.7)
- added R25: 105K, Resistor_SMD:R_0603_1608Metric_Pad0.98x0.95mm_HandSolder, F.Cu at (36.8, 21.7)
- added R26: 1k, common:R_0603, F.Cu at (35.3, 168.2)
- added R27: 1k, common:R_0603, F.Cu at (35.3, 170.8)
- added R28: 20k, common:R_0603, F.Cu at (35.3, 173.3)
- added R29: 43.2K, Resistor_SMD:R_0603_1608Metric_Pad0.98x0.95mm_HandSolder, F.Cu at (36.8, 24.2)
- added R3: 330, Resistor_SMD:R_0603_1608Metric_Pad0.98x0.95mm_HandSolder, F.Cu at (142.3, 106.6)
- added R30: 5.76K, Resistor_SMD:R_0603_1608Metric_Pad0.98x0.95mm_HandSolder, F.Cu at (36.8, 26.7)
- added R31: 1, Resistor_SMD:R_0603_1608Metric_Pad0.98x0.95mm_HandSolder, F.Cu at (36.8, 29.2)
- added R32: 1M, common:R_0603, F.Cu at (35.3, 175.8)
- added R33: 10K, Resistor_SMD:R_0603_1608Metric_Pad0.98x0.95mm_HandSolder, F.Cu at (268.5, 148.4)
- added R4: 330, Resistor_SMD:R_0603_1608Metric_Pad0.98x0.95mm_HandSolder, F.Cu at (142.3, 109.1)
- added R5: 4.7K, Resistor_SMD:R_0603_1608Metric_Pad0.98x0.95mm_HandSolder, F.Cu at (142.3, 111.6)
- added R6: 4.7K, Resistor_SMD:R_0603_1608Metric_Pad0.98x0.95mm_HandSolder, F.Cu at (142.3, 114.1)
- added R7: 1K, Resistor_SMD:R_0603_1608Metric_Pad0.98x0.95mm_HandSolder, F.Cu at (250.4, 50.3)
- added R8: 47, Resistor_SMD:R_0603_1608Metric_Pad0.98x0.95mm_HandSolder, F.Cu at (250.4, 52.8)
- added R9: 4.7K, Resistor_SMD:R_0603_1608Metric_Pad0.98x0.95mm_HandSolder, F.Cu at (250.4, 55.3)
- added SD1: ~, air_sens_foots:SD_SLOT, F.Cu at (256.8, 153.1)
- added SW1: SW_SPST, Connector_PinHeader_2.54mm:PinHeader_1x02_P2.54mm_Vertical, F.Cu at (156.0, 107.3)
- added SW2: SW_Push, switch:SW_Tactile3x2.5, F.Cu at (166.2, 100.3)
- added U1: ATmega328P-A, Package_QFP:TQFP-32_7x7mm_P0.8mm, F.Cu at (164.0, 110.7)
- added U4: TPS54302, Package_TO_SOT_SMD:TSOT-23-6_HandSoldering, F.Cu at (34.0, 41.2)
- added U5: AMS1117-3.3, Package_TO_SOT_SMD:SOT-223-3_TabPin2, F.Cu at (35.4, 34.7)
- added U7: NRF24L01, transceiver:NRF24L01_QFN20, F.Cu at (30.3, 185.3)
- added U8: RFX2401C, transceiver:RFX2401C_QFN16, F.Cu at (40.0, 188.6)
- added Y1: 8MHz, air_sens_foots:crys_osc_smd3225_4, F.Cu at (147.1, 114.4)
- added Y3: 16MHz, common:Crystal_3225, F.Cu at (24.1, 185.0)
