File: hardware/boards/vehicle/car/car.kicad_pcb (KiCad board)
At the start: 2 copper layers, 121 parts, among them J1 Conn_01x04_Socket, J10 Conn_02x03_Odd_Even, J2 Conn_01x05_Socket, J3 Conn_01x05_Socket, J4 Conn_01x05_Socket, J5 Conn_01x02_Socket, J6 SMA, J7 02x04, J8 Conn_01x04_Socket, J9 Conn_02x05_Odd_Even, M1 Motor_DC, M2 Motor_DC, Q1 FQP27P06, Q10 AO3400A, Q11 2N3904, Q12 2N3904, Q2 AO3400A, Q3 FQP27P06, Q4 AO3400A, Q5 2N3904, Q6 2N3904, Q7 FQP27P06, Q8 AO3400A, Q9 FQP27P06, SW1 SW_SPST, SW2 SW_Push, U1 ATmega328P-A, U4 TPS54302, U5 AMS1117-3.3, U7 NRF24L01, U8 RFX2401C, Y1 8MHz, Y3 16MHz

Commit message: pcb for car
Parts:
- removed R33: 10K, Resistor_SMD:R_0603_1608Metric_Pad0.98x0.95mm_HandSolder
- removed the SW1 at (156.0, 107.3)
- D10, D11, D4, D5, D6, D7, D8, D9: value UF5408 -> SS36; footprint Diode_THT:D_DO-201AD_P15.24mm_Horizontal -> Diode_SMD:D_SMA_Handsoldering
- moved C31 174.8 mm to (156.1, 67.7), turned to 180 degrees
- moved C30 171.9 mm to (156.1, 69.7), turned to 180 degrees
- moved Q4 170.3 mm to (143.8, 136.6), turned to 90 degrees
- moved U8 169.7 mm to (151.9, 61.0), turned to 180 degrees
- moved Y3 168.9 mm to (147.5, 69.6), turned to 90 degrees
- moved C37 168.0 mm to (146.7, 60.5), turned to -90 degrees
- moved C36 167.7 mm to (148.7, 60.5), turned to -90 degrees
- moved C38 167.0 mm to (142.7, 60.5), turned to -90 degrees
- moved C29 167.0 mm to (152.1, 70.1), turned to 180 degrees
- moved C33 166.1 mm to (156.1, 63.7), turned to 180 degrees
- moved R28 165.8 mm to (156.1, 59.7), turned to 180 degrees
- moved L7 164.9 mm to (156.1, 65.7)
- moved C28 164.1 mm to (152.1, 72.1), turned to 180 degrees
- moved C35 163.5 mm to (148.7, 64.1), turned to 90 degrees
- moved L8 163.3 mm to (151.3, 65.2), turned to 90 degrees
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- renumbered SW2 to SW1
Connections:
- BT1 pad 1: Net-(BT1-+) -> 12V
- J10 pad 1: 12V -> SD_CS
- J10 pad 2: GND -> MOSI
- J10 pad 3: MISO -> SCK
- J10 pad 4: SD_CS -> 3V3
- J10 pad 5: SCK -> MISO
- J10 pad 6: MOSI -> GND
Routing:
- net 3V3: track 0.00 -> 274.9 mm, vias 0 -> 14
- net GND: track 0.00 -> 229.7 mm, vias 0 -> 16
- net 12V: track 0.00 -> 210.8 mm, vias 0 -> 1
- net 5V: track 0.00 -> 110.9 mm, vias 0 -> 2
- net MOSI: track 0.00 -> 99.5 mm, vias 0 -> 4
- net SCK: track 0.00 -> 92.5 mm, vias 0 -> 4
- net MISO: track 0.00 -> 85.5 mm, vias 0 -> 4
- net M2_EN_CW: track 0.00 -> 65.2 mm, vias 0 -> 1
- net M2_EN_CCW: track 0.00 -> 64.5 mm, vias 0 -> 1
- net M1_EN_CCW: track 0.00 -> 62.8 mm
- net M1_EN_CW: track 0.00 -> 57.8 mm, vias 0 -> 1
- net RC_EN: track 0.00 -> 54.5 mm, vias 0 -> 2
- net SD_CS: track 0.00 -> 53.4 mm, vias 0 -> 2
- net RC_CS: track 0.00 -> 36.4 mm, vias 0 -> 1
- net M2_PWM_CCW: track 0.00 -> 35.3 mm, vias 0 -> 1
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- added copper zone on B.Cu, net GND
Other:
- board outline added: 50 x 95 mm
- board text added: "D4"
