File: hardware/boards/module/lidar/accelerometer.kicad_sch (KiCad schematic)
At the start: 6 parts, among them U2 BNO055, Y2 32.768kHz

Commit message: added all footprints for lidar and car
Parts:
- added J8: Conn_01x04_Socket, Connector_PinHeader_2.54mm:PinHeader_1x04_P2.54mm_Vertical, symbol Connector:Conn_01x04_Socket
- C10, C7, C8, C9: footprint (none) -> Capacitor_SMD:C_0603_1608Metric_Pad1.08x0.95mm_HandSolder
- U2: footprint Package_LGA:LGA-28_5.2x3.8mm_P0.5mm -> accelerometer:BNO055_Hand_Soldering_LGA-28_5.2x3.8mm_P0.5mm
- Y2: footprint (none) -> Crystal:Crystal_SMD_3215-2Pin_3.2x1.5mm
Connections:
- net 3V3: now also J8.3 (Pin_3)
- net GND: now also J8.4 (Pin_4)
- net RX: now also J8.2 (Pin_2)
- net TX: now also J8.1 (Pin_1)
Other:
- moved on the sheet: C10, C7, C8, C9, U2, Y2
