File: hardware/boards/module/lidar/lidar.kicad_sch (KiCad schematic)
At the start: 0 parts

Commit message: lidar schematic
Parts:
- added C1, C4, C6: 100nF, symbol Device:C
- added C2, C3: 12pF, symbol Device:C
- added C5: 10uF, symbol Device:C_Polarized
- added D1, D2: LED, symbol Device:LED
- added G1: ~, symbol air_sens_lib:module_gpio
- added J1: Conn_01x04_Socket, symbol Connector:Conn_01x04_Socket
- added J2: Lidar, symbol Connector:Conn_01x04_Socket
- added J3, J4, J5, J6: Conn_01x03_Socket, symbol Connector:Conn_01x03_Socket
- added J7: Conn_01x05_Socket, symbol Connector:Conn_01x05_Socket
- added Q1: AO3407A, symbol Simulation_SPICE:PMOS
- added R1, R4: 10K, symbol Device:R
- added R2, R3: 330, symbol Device:R
- added R5: 100, symbol Device:R
- added R6: 1K, symbol Device:R
- added SW1: SW_Push, symbol Switch:SW_Push
- added U1: ATmega128A-A, Package_QFP:TQFP-64_14x14mm_P0.8mm, symbol MCU_Microchip_ATmega:ATmega128A-A
- added Y1: 16MHz, symbol Device:Crystal_GND24
Connections:
- new net: D1.1 (K), R2.1
- new net: C3.1, U1.23 (XTAL2), Y1.3
- new net: C2.1, U1.24 (XTAL1), Y1.1
- new net: C4.2, U1.62 (AREF)
- new net: J2.2 (Pin_2), R6.2
- new net: C5.1, C6.1, J2.1 (Pin_1), Q1.1 (D)
- new net: C1.2, SW1.1
- new net: D2.1 (K), R3.1
- new net 3V3: C4.1, G1.1 (3V3), J1.3 (Pin_3), R1.1, U1.21 (VCC), U1.52 (VCC), U1.64 (AVCC)
- new net 5V: G1.2 (5V), J4.2 (Pin_2), J5.2 (Pin_2), J6.2 (Pin_2), Q1.3 (S), R4.2
- new net ADC0: J3.1 (Pin_1), U1.61 (PF0)
- new net ADC1: J3.2 (Pin_2), U1.60 (PF1)
- new net ADC2: J3.3 (Pin_3), U1.59 (PF2)
- new net D1: D1.2 (A), U1.31 (PD6)
- new net D2: D2.2 (A), U1.32 (PD7)
- new net DEBUG_0: J7.1 (Pin_1), U1.10 (PB0)
- new net DEBUG_1: J7.2 (Pin_2), U1.11 (PB1)
- new net DEBUG_2: J7.3 (Pin_3), U1.12 (PB2)
- new net DEBUG_3: J7.4 (Pin_4), U1.13 (PB3)
- new net DEBUG_4: J7.5 (Pin_5), U1.14 (PB4)
- new net GND: C1.1, C2.2, C3.2, C5.2, C6.2, G1.3 (GND), J1.4 (Pin_4), J2.3 (Pin_3), J4.1 (Pin_1), J5.1 (Pin_1), J6.1 (Pin_1), Q1.2 (G), R2.2, R3.2, R4.1, R5.2, U1.22 (GND), U1.53 (GND), U1.63 (GND), Y1.2, Y1.4
- new net LIDAR_EN: R5.1, U1.16 (PB6)
- new net LIDAR_PWM: J2.4 (Pin_4), U1.15 (PB5)
- new net RST: R1.2, SW1.2, U1.20 (~{RESET})
- new net RX0: J1.1 (Pin_1), R6.1, U1.2 (PE0)
- new net RX1: U1.27 (PD2)
- new net SCL: G1.5 (SCL), U1.25 (PD0)
- new net SDA: G1.4 (SDA), U1.26 (PD1)
- new net SERVO_A_PWM: J4.3 (Pin_3), U1.5 (PE3)
- new net SERVO_B_PWM: J5.3 (Pin_3), U1.6 (PE4)
- new net SERVO_C_PWM: J6.3 (Pin_3), U1.7 (PE5)
- new net TX0: J1.2 (Pin_2), U1.3 (PE1)
- new net TX1: U1.28 (PD3)
- no-connect marks 0 -> 33
Other:
- added sheet Accelerometer (accelerometer.kicad_sch)

Commit message: added all footprints for lidar and car
Parts:
- C1, C2, C3, C4, C6: footprint (none) -> Capacitor_SMD:C_0603_1608Metric_Pad1.08x0.95mm_HandSolder
- C5: footprint (none) -> Capacitor_THT:CP_Radial_D5.0mm_P2.00mm
- D1, D2: footprint (none) -> LED_SMD:LED_0603_1608Metric_Pad1.05x0.95mm_HandSolder
- G1, J7: footprint (none) -> Connector_PinHeader_2.54mm:PinHeader_1x05_P2.54mm_Vertical
- J1, J2: footprint (none) -> Connector_PinHeader_2.54mm:PinHeader_1x04_P2.54mm_Vertical
- J3, J4, J5, J6: footprint (none) -> Connector_PinHeader_2.54mm:PinHeader_1x03_P2.54mm_Vertical
- Q1: footprint (none) -> Package_TO_SOT_SMD:TSOT-23-6_HandSoldering
- R1, R2, R3, R4, R5, R6: footprint (none) -> Resistor_SMD:R_0603_1608Metric_Pad0.98x0.95mm_HandSolder
- SW1: footprint (none) -> switch:SW_Tactile3x2.5
- Y1: value 16MHz -> 8MHz; footprint (none) -> air_sens_foots:crys_osc_smd3225_4
Changed lines of the file:
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@@
 			)
 		)
-		(property "Footprint" ""
+		(property "Footprint" "Connector_PinHeader_2.54mm:PinHeader_1x03_P2.54mm_Vertical"
 			(at 173.99 129.54 0)
 			(effects
@@
 			)
 		)
-		(property "Footprint" ""
+		(property "Footprint" "LED_SMD:LED_0603_1608Metric_Pad1.05x0.95mm_HandSolder"
 			(at 229.87 139.7 0)
 			(effects
@@
 			)
 		)
-		(property "Footprint" ""
+		(property "Footprint" "Connector_PinHeader_2.54mm:PinHeader_1x03_P2.54mm_Vertical"
 			(at 267.97 35.56 0)
 			(effects
@@
 			)
 		)
-		(property "Footprint" ""
+		(property "Footprint" "Connector_PinHeader_2.54mm:PinHeader_1x03_P2.54mm_Vertical"
 			(at 173.99 140.97 0)
 			(effects
@@
 			)
 		)
-		(property "Footprint" ""
+		(property "Footprint" "Connector_PinHeader_2.54mm:PinHeader_1x05_P2.54mm_Vertical"
 			(at 242.57 36.83 0)
 			(effects
@@
 			)
 		)
-		(property "Footprint" ""
+		(property "Footprint" "Resistor_SMD:R_0603_1608Metric_Pad0.98x0.95mm_HandSolder"
 			(at 248.92 105.918 90)
 			(effects
@@
 			)
 		)
-		(property "Footprint" ""
+		(property "Footprint" "Connector_PinHeader_2.54mm:PinHeader_1x04_P2.54mm_Vertical"
 			(at 186.69 38.1 0)
 			(effects
@@
 			)
 		)
-		(property "Footprint" ""
+		(property "Footprint" "Connector_PinHeader_2.54mm:PinHeader_1x04_P2.54mm_Vertical"
 			(at 257.81 104.14 0)
 			(effects
@@
 			)
 		)
-		(property "Footprint" ""
+		(property "Footprint" "Capacitor_SMD:C_0603_1608Metric_Pad1.08x0.95mm_HandSolder"
 			(at 58.42 106.9848 0)
 			(effects
@@
 			)
 		)
-		(property "Value" "16MHz"
-			(at 39.37 94.234 90)
+		(property "Value" "8MHz"
+			(at 37.338 94.234 90)
 			(effects
 				(font
@@
 			)
 		)
-		(property "Footprint" ""
+		(property "Footprint" "air_sens_foots:crys_osc_smd3225_4"
 			(at 34.29 97.79 0)
 			(effects
@@
 			)
 		)
-		(property "Footprint" ""
+		(property "Footprint" "switch:SW_Tactile3x2.5"
 			(at 91.44 38.1 0)
 			(effects
@@
 			)
 		)
-		(property "Footprint" ""
+		(property "Footprint" "Package_TO_SOT_SMD:TSOT-23-6_HandSoldering"
 			(at 238.76 86.36 0)
 			(effects
@@
 			)
 		)
-		(property "Footprint" ""
+		(property "Footprint" "Capacitor_THT:CP_Radial_D5.0mm_P2.00mm"
 			(at 239.7252 96.52 0)
 			(effects
@@
 			)
 		)
-		(property "Footprint" ""
+		(property "Footprint" "Resistor_SMD:R_0603_1608Metric_Pad0.98x0.95mm_HandSolder"
 			(at 97.282 36.83 90)
 			(effects
@@
 			)
 		)
-		(property "Footprint" ""
+		(property "Footprint" "Resistor_SMD:R_0603_1608Metric_Pad0.98x0.95mm_HandSolder"
 			(at 237.49 149.098 90)
 			(effects
@@
 			)
 		)
-		(property "Footprint" ""
+		(property "Footprint" "Connector_PinHeader_2.54mm:PinHeader_1x03_P2.54mm_Vertical"
 			(at 173.99 152.4 0)
 			(effects
@@
 			)
 		)
-		(property "Footprint" ""
+		(property "Footprint" "Connector_PinHeader_2.54mm:PinHeader_1x05_P2.54mm_Vertical"
 			(at 35.56 57.15 0)
 			(effects
@@
 			)
 		)
-		(property "Footprint" ""
+		(property "Footprint" "Capacitor_SMD:C_0603_1608Metric_Pad1.08x0.95mm_HandSolder"
 			(at 24.13 101.9048 0)
 			(effects
@@
 			)
 		)
-		(property "Footprint" ""
+		(property "Footprint" "Resistor_SMD:R_0603_1608Metric_Pad0.98x0.95mm_HandSolder"
 			(at 222.25 85.598 90)
 			(effects
@@
 			)
 		)
-		(property "Footprint" ""
+		(property "Footprint" "Capacitor_SMD:C_0603_1608Metric_Pad1.08x0.95mm_HandSolder"
 			(at 86.36 42.2148 0)
 			(effects
@@
 			)
 		)
-		(property "Footprint" ""
+		(property "Footprint" "Capacitor_SMD:C_0603_1608Metric_Pad1.08x0.95mm_HandSolder"
 			(at 24.13 91.7448 0)
 			(effects
@@
 			)
 		)
-		(property "Footprint" ""
+		(property "Footprint" "LED_SMD:LED_0603_1608Metric_Pad1.05x0.95mm_HandSolder"
 			(at 229.87 147.32 0)
 			(effects
@@
 			)
 		)
-		(property "Footprint" ""
+		(property "Footprint" "Resistor_SMD:R_0603_1608Metric_Pad0.98x0.95mm_HandSolder"
 			(at 229.87 80.518 90)
 			(effects
@@
 			)
 		)
-		(property "Footprint" ""
+		(property "Footprint" "Resistor_SMD:R_0603_1608Metric_Pad0.98x0.95mm_HandSolder"
 			(at 237.49 141.478 90)
 			(effects
@@
 			)
 		)
-		(property "Footprint" ""
+		(property "Footprint" "Capacitor_SMD:C_0603_1608Metric_Pad1.08x0.95mm_HandSolder"
 			(at 247.3452 96.52 0)
 			(effects

Commit message: lidar pcb
Parts:
- removed Q1: AO3407A, Package_TO_SOT_SMD:TSOT-23-6_HandSoldering, symbol Simulation_SPICE:PMOS
- added Q1: AO3401A, Package_TO_SOT_SMD:SOT-23_Handsoldering, symbol Transistor_FET:AO3401A
Connections:
- net 5V: now also Q1.2 (S)
- net GND: now also Q1.1 (G)
- net at C5.1, C6.1, J2.1 (Pin_1): now also Q1.3 (D)
Changed lines of the file:
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@@
 	)
 	(junction
-		(at 236.22 78.74)
-		(diameter 0)
-		(color 0 0 0 0)
-	)
-	(junction
 		(at 226.06 99.06)
 		(diameter 0)
@@
 	)
 	(junction
+		(at 236.22 78.74)
+		(diameter 0)
+		(color 0 0 0 0)
+	)
+	(junction
 		(at 162.56 140.97)
 		(diameter 0)
@@
 	)
 	(symbol
+		(lib_id "Transistor_FET:AO3401A")
+		(at 233.68 83.82 0)
+		(mirror x)
+		(unit 1)
+		(exclude_from_sim no)
+		(in_bom yes)
+		(on_board yes)
+		(dnp no)
+		(property "Reference" "Q1"
+			(at 238.252 82.55 0)
+			(effects
+				(font
+					(size 1.27 1.27)
+				)
+				(justify left)
+			)
+		)
+		(property "Value" "AO3401A"
+			(at 238.252 84.328 0)
+			(effects
+				(font
+					(size 1.27 1.27)
+				)
+				(justify left)
+			)
+		)
+		(property "Footprint" "Package_TO_SOT_SMD:SOT-23_Handsoldering"
+			(at 238.76 81.915 0)
+			(effects
+				(font
+					(size 1.27 1.27)
+					(italic yes)
+				)
+				(justify left)
+				(hide yes)
+			)
+		)
+		(property "Datasheet" "http://www.aosmd.com/pdfs/datasheet/AO3401A.pdf"
+			(at 238.76 80.01 0)
+			(effects
+				(font
+					(size 1.27 1.27)
+				)
+				(justify left)
+				(hide yes)
+			)
+		)
+		(property "Description" "-4.0A Id, -30V Vds, P-Channel MOSFET, SOT-23"
+			(at 233.68 83.82 0)
+			(effects
+				(font
+					(size 1.27 1.27)
+				)
+				(hide yes)
+			)
+		)
+		(pin "3"
+		)
+		(pin "1"
+		)
+		(pin "2"
+		)
+		(instances
+			(project ""
+				(path "/ddbee91c-d870-4cea-baff-6659bab9b5fd"
+					(reference "Q1")
+					(unit 1)
+				)
+			)
+		)
+	)
+	(symbol
 		(lib_id "Connector:Conn_01x03_Socket")
 		(at 173.99 140.97 0)
@@
 					(unit 1)
 				)
-			)
-		)
-	)
-	(symbol
-		(lib_id "Simulation_SPICE:PMOS")
-		(at 233.68 83.82 0)
-		(mirror x)
-		(unit 1)
-		(exclude_from_sim no)
-		(in_bom yes)
-		(on_board yes)
-		(dnp no)
-		(property "Reference" "Q1"
-			(at 238.252 82.296 0)
-			(effects
-				(font
-					(size 1.27 1.27)
-				)
-				(justify left)
-			)
-		)
-		(property "Value" "AO3407A"
-			(at 238.506 84.074 0)
-			(effects
-				(font
-					(size 1.27 1.27)
-				)
-				(justify left)
-			)
-		)
-		(property "Footprint" "Package_TO_SOT_SMD:TSOT-23-6_HandSoldering"
-			(at 238.76 86.36 0)
-			(effects
-				(font
-					(size 1.27 1.27)
-				)
-				(hide yes)
-			)
-		)
-		(property "Datasheet" "https://ngspice.sourceforge.io/docs/ngspice-html-manual/manual.xhtml#cha_MOSFETs"
-			(at 233.68 71.12 0)
-			(effects
-				(font
-					(size 1.27 1.27)
-				)
-				(hide yes)
-			)
-		)
-		(property "Description" "P-MOSFET transistor, drain/source/gate"
-			(at 233.68 83.82 0)
-			(effects
-				(font
-					(size 1.27 1.27)
-				)
-				(hide yes)
-			)
-		)
-		(property "Sim.Device" "PMOS"
-			(at 233.68 66.675 0)
-			(effects
-				(font
-					(size 1.27 1.27)
-				)
-				(hide yes)
-			)
-		)
-		(property "Sim.Type" "VDMOS"
-			(at 233.68 64.77 0)
-			(effects
-				(font
-					(size 1.27 1.27)
-				)
-				(hide yes)
-			)
-		)
-		(property "Sim.Pins" "1=D 2=G 3=S"
-			(at 233.68 68.58 0)
-			(effects
-				(font
-					(size 1.27 1.27)
-				)
-				(hide yes)
-			)
-		)
-		(pin "1"
-		)
-		(pin "3"
-		)
-		(pin "2"
-		)
-		(instances
-			(project ""
-				(path "/ddbee91c-d870-4cea-baff-6659bab9b5fd"
-					(reference "Q1")
-					(unit 1)
-				)
