File: kicad/schematic/controller/controller.kicad_pcb (KiCad board)
At the start: 2 copper layers, 187 x 104.5 mm, 79 parts, among them J1 01x02, J10 01x05, J11 01x03, J2 01x06, J3 01x06, J4 01x02, J6 SMA, J7 02x04, J8 01x03, J9 01x05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

Commit message: update gerber file
Routing:
- net +3.3V: track 232.8 -> 239.8 mm, vias 4 -> 6
- net Net-(D2-A): track 49.6 -> 54.8 mm
- net +5V: track 460.2 -> 463.0 mm, vias 3 -> 4
- net SCK: track 192.7 -> 194.8 mm, vias 5 -> 8
- net MISO: track 198.3 -> 199.6 mm, vias 5 -> 9
- net RXD: track 43.5 -> 44.6 mm
- net TXD: track 41.8 -> 42.8 mm
- net Net-(U1-PC4/ADC4/SDA/PCINT12): track 70.8 -> 70.9 mm, vias 1 -> 2
- net MOSI: vias 5 -> 9
