File: kicad/schematic/controller/controller.kicad_pcb (KiCad board)
At the start: 2 copper layers, 86.3 x 52 mm, 76 parts, among them J1 01x02, J2 01x06, J3 01x06, J4 01x02, J5 01x06, J6 SMA, J7 02x04, J8 01x03, SW1 Reset, SW2 Power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

Commit message: feat(pcb): working pcb design
Parts:
- removed J5: 01x06, connector:Pin_01x06
- added J10: 01x05, connector:Pin_01x05, F.Cu at (215.2, 113.8)
- added J11: 01x03, connector:Pin_01x03, F.Cu at (138.0, 121.5)
- added J9: 01x05, connector:Pin_01x05, F.Cu at (97.0, 112.2)
- added R1: 1M, common:R_0603, F.Cu at (98.8, 59.4)
- SW1: footprint common:SW_Tactile06x06 -> switch:SW_Tactile3x2.5
- SW2: footprint common:SW_Slide -> switch:SW_Slide9.1x3.5
- SW4, SW5: value SW_Push -> SW; footprint common:SW_Tactile12x12 -> switch:SW_Tactile12x12
- moved U9 156.7 mm to (214.6, 126.2), turned to 90 degrees
- moved U10 143.3 mm to (92.4, 125.1), turned to 90 degrees
- moved C24 126.5 mm to (201.3, 107.1), turned to 180 degrees
- moved SW1 116.2 mm to (197.8, 105.2)
- moved R16 112.4 mm to (201.2, 103.3), turned to 0 degrees
- moved R11 111.7 mm to (161.7, 68.5), turned to 180 degrees
- moved R12 109.8 mm to (161.7, 70.7), turned to 180 degrees
- moved R13 109.2 mm to (161.7, 73.5), turned to 180 degrees
- moved R14 108.5 mm to (161.7, 76.2), turned to 180 degrees
- moved R15 107.7 mm to (161.7, 78.8), turned to 180 degrees
- moved C26 102.4 mm to (101.7, 49.6), turned to -90 degrees
- moved R26 101.6 mm to (112.2, 59.7)
- moved C34 101.0 mm to (115.0, 50.3)
- moved J4 100.3 mm to (154.5, 83.8), turned to 90 degrees
- moved C25 99.8 mm to (100.1, 49.6), turned to -90 degrees
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Connections:
- J3 pad 1: Net-(U4-T_CLK) -> GND
- J3 pad 2: Net-(U4-T_CS) -> Net-(U4-T_CLK)
- J3 pad 3: Net-(U4-T_DIN) -> Net-(U4-T_CS)
- J3 pad 4: Net-(U4-T_DO) -> Net-(U4-T_DIN)
- J3 pad 5: Net-(U4-T_IRQ) -> Net-(U4-T_DO)
- J3 pad 6: GND -> Net-(U4-T_IRQ)
- R18 pad 1: Net-(U1-PCINT20/XCK/T0/PD4) -> Net-(U1-PC2/ADC2/PCINT10)
- R19 pad 1: Net-(U1-PCINT21/OC0B/T1/PD5) -> Net-(U1-PC3/ADC3/PCINT11)
- R20 pad 1: Net-(U1-PCINT19/OC2B/INT1/PD3) -> Net-(U1-PCINT20/XCK/T0/PD4)
- R21 pad 1: Net-(U1-INT0/PCINT18/PD2) -> Net-(U1-PCINT19/OC2B/INT1/PD3)
- SW1 pad 2: (no net) -> DTR
- SW3 pad 1: Net-(U1-PCINT20/XCK/T0/PD4) -> Net-(U1-PC2/ADC2/PCINT10)
- SW3 pad 3: Net-(U1-PCINT21/OC0B/T1/PD5) -> Net-(U1-PC3/ADC3/PCINT11)
- SW4 pad 1: Net-(U1-PCINT19/OC2B/INT1/PD3) -> Net-(U1-PCINT20/XCK/T0/PD4)
- SW4 pad 2: (no net) -> unconnected-(SW4-Pad2)
- SW4 pad 4: (no net) -> unconnected-(SW4-Pad4)
- SW5 pad 1: Net-(U1-INT0/PCINT18/PD2) -> Net-(U1-PCINT19/OC2B/INT1/PD3)
- SW5 pad 2: (no net) -> unconnected-(SW5-Pad2)
- SW5 pad 4: (no net) -> unconnected-(SW5-Pad4)
- U1 pad 23: Net-(U1-PC0/ADC0/PCINT8) -> JOY1-X
- U1 pad 24: Net-(U1-PC1/ADC1/PCINT9) -> JOY1-Y
- U1 pad 26: Net-(D2-A) -> Net-(U1-PC3/ADC3/PCINT11)
- U1 pad 32: Net-(U1-INT0/PCINT18/PD2) -> JOY1-B
- U1 pad 9: Net-(U1-PCINT21/OC0B/T1/PD5) -> Net-(D2-A)
- U7 pad 21: (no net) -> GND
Routing:
- net +5V: track 40.9 -> 458.7 mm, vias 0 -> 3
- net MOSI: track 0.00 -> 208.2 mm, vias 0 -> 5
- net +3.3V: track 30.3 -> 231.3 mm, vias 0 -> 4
- net MISO: track 0.00 -> 198.8 mm, vias 0 -> 4
- net SCK: track 0.00 -> 192.7 mm, vias 0 -> 5
- net CE: track 0.00 -> 144.1 mm, vias 0 -> 5
- net CSN: track 0.00 -> 135.5 mm, vias 0 -> 4
- net Net-(U1-PC5/ADC5/SCL/PCINT13): track 0.00 -> 122.2 mm
- net GND: track 0.00 -> 122.2 mm, vias 0 -> 28
- net Net-(U1-ADC7): track 0.00 -> 119.2 mm, vias 0 -> 1
- net Net-(U1-ADC6): track 0.00 -> 113.2 mm, vias 0 -> 1
- net Net-(U1-PC2/ADC2/PCINT10): track 0.00 -> 105.2 mm
- net Net-(U1-PC3/ADC3/PCINT11): track 0.00 -> 98.9 mm
- net Net-(U1-PC4/ADC4/SDA/PCINT12): track 0.00 -> 70.8 mm, vias 0 -> 1
- net JOY1-Y: track 0.00 -> 67.1 mm, vias 0 -> 2
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- added copper zone on B.Cu, net GND
Other:
- board size 86.3 x 52 mm -> 187 x 104.5 mm

Commit message: update controller pcb
Routing:
- net GND: track 122.2 -> 132.0 mm, vias 28 -> 138
- net +3.3V: track 231.3 -> 232.8 mm
- net +5V: track 458.7 -> 460.2 mm
- net MISO: track 198.8 -> 198.3 mm, vias 4 -> 5
Other:
- board text added: "+"
- board text added: "-"
- board text added: "3.3V"
- board text added: "3.3V|CSN|MOSI|IRQ"
- board text added: "5V"
- board text added: "GND"
- board text added: "GND|CE|SCK|MISO"
- board text added: "GND|GND|5V|RXD|TXD|DTR"
- board text added: "Project VEMAR Version 1.0.0"
- board text added: "SCK|MISO|MOSI"
- board text added: "T_CLK"
- board text added: "T_CS"
- board text added: "T_DIN"
- board text added: "T_DO"
- board text added: "T_IRQ"

Commit message: update gerber file
Parts:
- added R2: 10k, common:R_0603, F.Cu at (189.7, 113.8)
- added R3: 10k, common:R_0603, F.Cu at (88.7, 107.2)
- C2, C28, C29, C3: value 22pF -> 12pF
- D2: value ~ -> Green
Connections:
- net Net-(U1-ADC6) renamed JOY2-X
- net Net-(U1-ADC7) renamed JOY2-Y
- net Net-(U1-PC5/ADC5/SCL/PCINT13) renamed JOY2-B
Routing:
- net +5V: track 460.2 -> 471.4 mm, vias 3 -> 4
- net +3.3V: track 232.8 -> 239.8 mm, vias 4 -> 6
- net Net-(D2-A): track 49.6 -> 54.8 mm
- net JOY2-B: track 122.2 -> 124.6 mm
- net SCK: track 192.7 -> 194.8 mm, vias 5 -> 8
- net MISO: track 198.3 -> 199.6 mm, vias 5 -> 9
- net RXD: track 43.5 -> 44.6 mm
- net TXD: track 41.8 -> 42.8 mm
- net Net-(U1-PC4/ADC4/SDA/PCINT12): track 70.8 -> 70.9 mm, vias 1 -> 2
- net MOSI: vias 5 -> 9
