File: kicad/schematic/controller/controller.kicad_sch (KiCad schematic)
At the start: 25 parts, among them J10 01x05, J11 01x03, J2 01x06, J7 02x04, J9 01x05, SW1 Reset, SW3 SW_SPDT, SW4 SW, SW5 SW, U1 ATmega328P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

Commit message: update controller pcb
Parts:
- C1, C24: Ext. Price (none) -> 0.19; LCSC Part (none) -> C14663; Manufacturer (none) -> YAGEO; Manufacturer Part (none) -> CC0603KRX7R9BB104; Unit Price (none) -> 0.0019
- C2, C3: value 22pF -> 12pF; Ext. Price (none) -> 0.27; LCSC Part (none) -> C107034; Manufacturer (none) -> YAGEO; Manufacturer Part (none) -> CC0603JRNPO9BN120; Unit Price (none) -> 0.0027
- D2: value ~ -> Green; Ext. Price (none) -> 0.49; LCSC Part (none) -> C19273151; Manufacturer (none) -> YONGYUTAI; Manufacturer Part (none) -> YLED0603G; Unit Price (none) -> 0.0049
- R16, R18, R19, R20, R21: Ext. Price (none) -> 0.08; LCSC Part (none) -> C2906982; Manufacturer (none) -> FOJAN; Manufacturer Part (none) -> FRC0603F1002TS; Unit Price (none) -> 0.0008
- R22: Ext. Price (none) -> 0.08; LCSC Part (none) -> C2907152; Manufacturer (none) -> FOJAN; Manufacturer Part (none) -> FRC0603J331 TS; Unit Price (none) -> 0.0008
- RV1: Ext. Price (none) -> 1.35; LCSC Part (none) -> C17444183; Manufacturer (none) -> BOURNS; Manufacturer Part (none) -> PTA4543-2015DPB103; Unit Price (none) -> 1.3457
- SW1: Ext. Price (none) -> 0.36; LCSC Part (none) -> C49234121; Manufacturer (none) -> hanxia; Manufacturer Part (none) -> HX-B3U-1000P-1.6N; Unit Price (none) -> 0.0712
- SW3: Ext. Price (none) -> 3.49; LCSC Part (none) -> AliExpress; Manufacturer (none) -> SWITCHES; Manufacturer Part (none) -> MST103; Unit Price (none) -> 3.49
- SW4, SW5: Ext. Price (none) -> 0.53; LCSC Part (none) -> C19077684; Manufacturer (none) -> Yuandi; Manufacturer Part (none) -> TS-1094TS-B3D2-T-Y; Unit Price (none) -> 0.1068
- U1: Ext. Price (none) -> 1.72; LCSC Part (none) -> C14877; Manufacturer (none) -> MICROCHIP; Manufacturer Part (none) -> ATMEGA328P-AU; Unit Price (none) -> 1.7203
- U10, U9: Ext. Price (none) -> 2.47; LCSC Part (none) -> AliExpress; Manufacturer (none) -> -; Manufacturer Part (none) -> Hall-Effect Joysticks; Unit Price (none) -> 2.47
- Y1: Ext. Price (none) -> 0.59; LCSC Part (none) -> C13738; Manufacturer (none) -> YXC Crystal Oscillators; Manufacturer Part (none) -> X322516MLB4SI; Unit Price (none) -> 0.059

Commit message: update gerber file
Parts:
- added R2, R3: 10k, common:R_0603, symbol common:Resistor
Connections:
- net +5V: now also R2.2, R3.2
- net JOY1-B: now also R2.1
- net JOY2-B: now also R3.1
