File: kicad/schematic/controller/power.kicad_sch (KiCad schematic)
At the start: 12 parts, among them J8 01x03, U2 AMS1117-5.0, U3 AMS1117-3.3

Commit message: feat(pcb): pcb wip
Parts:
- removed BT1: Battery, symbol common:Battery
- D1: value ~ -> Red
- D3: footprint (none) -> common:D_SOD123
- J1: value ~ -> 01x02; footprint (none) -> connector:Pin_01x02
- J8: footprint (none) -> connector:Pin_01x03
- SW2: value ~ -> Power; footprint (none) -> common:SW_Slide
Changed lines of the file:
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@@
-	)
-	(junction
-		(at 76.2 78.74)
-		(diameter 0)
-		(color 0 0 0 0)
 	)
 	(junction
@@
 	)
 	(junction
-		(at 76.2 68.58)
-		(diameter 0)
-		(color 0 0 0 0)
-	)
-	(junction
 		(at 116.84 68.58)
 		(diameter 0)
@@
 	(wire
 		(pts
-			(xy 76.2 60.96) (xy 76.2 68.58)
-		)
-		(stroke
-			(width 0)
-			(type default)
-		)
-	)
-	(wire
-		(pts
 			(xy 148.59 68.58) (xy 163.83 68.58)
 		)
@@
 	(wire
 		(pts
-			(xy 53.34 64.77) (xy 53.34 60.96)
-		)
-		(stroke
-			(width 0)
-			(type default)
-		)
-	)
-	(wire
-		(pts
 			(xy 93.98 96.52) (xy 93.98 106.68)
 		)
@@
 	(wire
 		(pts
-			(xy 76.2 71.12) (xy 76.2 78.74)
-		)
-		(stroke
-			(width 0)
-			(type default)
-		)
-	)
-	(wire
-		(pts
-			(xy 53.34 74.93) (xy 53.34 78.74)
-		)
-		(stroke
-			(width 0)
-			(type default)
-		)
-	)
-	(wire
-		(pts
 			(xy 116.84 68.58) (xy 109.22 68.58)
 		)
@@
 	(wire
 		(pts
-			(xy 76.2 81.28) (xy 76.2 78.74)
+			(xy 76.2 71.12) (xy 76.2 81.28)
 		)
 		(stroke
@@
 		(pts
 			(xy 116.84 105.41) (xy 116.84 106.68)
-		)
-		(stroke
-			(width 0)
-			(type default)
-		)
-	)
-	(wire
-		(pts
-			(xy 53.34 60.96) (xy 76.2 60.96)
-		)
-		(stroke
-			(width 0)
-			(type default)
-		)
-	)
-	(wire
-		(pts
-			(xy 53.34 78.74) (xy 76.2 78.74)
 		)
 		(stroke
@@
 			)
 		)
-		(property "Footprint" ""
+		(property "Footprint" "common:D_SOD123"
 			(at 105.41 68.58 0)
 			(effects
@@
 			)
 		)
-		(property "Value" "~"
+		(property "Value" "01x02"
 			(at 72.39 73.35 0)
 			(effects
@@
 			)
 		)
-		(property "Footprint" ""
+		(property "Footprint" "connector:Pin_01x02"
 			(at 72.39 69.85 0)
 			(effects
@@
 			)
 		)
-		(property "Value" "~"
+		(property "Value" "Power"
 			(at 85.09 63.5 0)
 			(effects
@@
 			)
 		)
-		(property "Footprint" ""
+		(property "Footprint" "common:SW_Slide"
 			(at 85.09 68.58 0)
 			(effects
@@
 	)
 	(symbol
-		(lib_id "common:Battery")
-		(at 53.34 69.85 270)
+		(lib_id "common:LED")
+		(at 93.98 76.2 90)
 		(unit 1)
 		(exclude_from_sim no)
@@
 		(dnp no)
 		(fields_autoplaced yes)
-		(property "Reference" "BT1"
-			(at 57.15 67.3849 90)
-			(effects
-				(font
-					(size 1.27 1.27)
-				)
-				(justify left)
-			)
-		)
-		(property "Value" "Battery"
-			(at 57.15 69.9249 90)
-			(effects
-				(font
-					(size 1.27 1.27)
-				)
-				(justify left)
-			)
-		)
-		(property "Footprint" ""
-			(at 53.34 69.85 0)
-			(effects
-				(font
-					(size 1.27 1.27)
-				)
-				(hide yes)
-			)
-		)
-		(property "Datasheet" ""
-			(at 53.34 69.85 0)
-			(effects
-				(font
-					(size 1.27 1.27)
-				)
-				(hide yes)
-			)
-		)
-		(property "Description" "Multiple-Cell Battery"
-			(at 47.34 69.85 0)
-			(effects
-				(font
-					(size 1.27 1.27)
-				)
-				(hide yes)
-			)
-		)
-		(pin "1"
-		)
-		(pin "2"
-		)
-		(instances
-			(project "controller"
-				(path "/beaf00ba-d60c-407c-adfe-9d518bae0b16/c4e35d3f-6040-4882-878d-1a95fa713f03"
-					(reference "BT1")
-					(unit 1)
-				)
-			)
-		)
-	)
-	(symbol
-		(lib_id "common:LED")
-		(at 93.98 76.2 90)
-		(unit 1)
-		(exclude_from_sim no)
-		(in_bom yes)
-		(on_board yes)
-		(dnp no)
-		(fields_autoplaced yes)
 		(property "Reference" "D1"
 			(at 97.79 76.4549 90)
@@
 			)
 		)
-		(property "Value" "~"
+		(property "Value" "Red"
 			(at 93.98 76.2 0)
 			(effects
@@
 			)
 		)
-		(property "Footprint" ""
+		(property "Footprint" "connector:Pin_01x03"
 			(at 167.64 68.58 0)
 			(effects

Commit message: feat(schematic): cleanup controller
Parts:
- SW2: footprint common:SW_Slide -> switch:SW_Slide9.1x3.5

Commit message: update controller pcb
Parts:
- C4: Ext. Price (none) -> 0.39; LCSC Part (none) -> C3151830; Manufacturer (none) -> ROQANG; Manufacturer Part (none) -> RVT1V101M0605; Unit Price (none) -> 0.0393
- C5, C6: Ext. Price (none) -> 0.57; LCSC Part (none) -> C72505; Manufacturer (none) -> ROQANG; Manufacturer Part (none) -> RVT1H220M0605; Unit Price (none) -> 0.0283
- D1: Ext. Price (none) -> 0.51; LCSC Part (none) -> C19171390; Manufacturer (none) -> YONGYUTAI; Manufacturer Part (none) -> YLED0603R; Unit Price (none) -> 0.0051
- D3: Ext. Price (none) -> 0.20; LCSC Part (none) -> C2892681; Manufacturer (none) -> YONGYUTAI; Manufacturer Part (none) -> 1N4007; Unit Price (none) -> 0.004
- R17: Ext. Price (none) -> 0.07; LCSC Part (none) -> C2907113; Manufacturer (none) -> FOJAN; Manufacturer Part (none) -> FRC0603J102 TS; Unit Price (none) -> 0.0007
- SW2: Ext. Price (none) -> 0.34; LCSC Part (none) -> C49023767; Manufacturer (none) -> SHOU HAN; Manufacturer Part (none) -> MST-12D18G4 SPDT Slide Switch; Unit Price (none) -> 0.0677
- U2: Ext. Price (none) -> 0.32; LCSC Part (none) -> C347222; Manufacturer (none) -> UMW; Manufacturer Part (none) -> AMS1117-3.3; Unit Price (none) -> 0.0315
- U3: Ext. Price (none) -> 0.32; LCSC Part (none) -> C347223; Manufacturer (none) -> UMW; Manufacturer Part (none) -> AMS1117-5.0; Unit Price (none) -> 0.0315
