File: hardware/boards/controller/controller.kicad_sch (KiCad schematic)
At the start: 27 parts, among them J10 01x05, J11 01x03, J2 01x06, J7 02x04, J9 01x05, SW1 Reset, SW3 SW_SPDT, SW4 SW, SW5 SW, U1 ATmega328P, U10 Joystick, U9 Joystick, Y1 16MHz

Commit message: new version for pcb controller
Parts:
- removed J10, J9: 01x05, connector:Pin_01x05, symbol connector:Pin_01x05
- added C1: 1uF, common:C_0603, symbol common:Capacitor
- added C2: 100nF, common:C_0603, symbol common:Capacitor
- C3: renamed from C24; Ext. Price 0.19 -> 0.25; Unit Price 0.0019 -> 0.0025
- C4: renamed from C1; Ext. Price 0.19 -> 0.25; Unit Price 0.0019 -> 0.0025
- J1: renamed from J11; now left out of the parts list
- J2: now left out of the parts list
- J3: renamed from J7; now left out of the parts list
- R1: renamed from R16; Ext. Price 0.08 -> 0.10; Unit Price 0.0008 -> 0.001
- R2: renamed from R18; Ext. Price 0.08 -> 0.10; Unit Price 0.0008 -> 0.001
- R3: renamed from R19; Ext. Price 0.08 -> 0.10; Unit Price 0.0008 -> 0.001
- R4: renamed from R21; Ext. Price 0.08 -> 0.10; Unit Price 0.0008 -> 0.001
- R5: renamed from R20; Ext. Price 0.08 -> 0.10; Unit Price 0.0008 -> 0.001
- R7: renamed from R2; Ext. Price (none) -> 0.10; LCSC Part (none) -> C2906982; Manufacturer (none) -> FOJAN; Manufacturer Part (none) -> FRC0603F1002TS; Unit Price (none) -> 0.001
- R8: renamed from R3; Ext. Price (none) -> 0.10; LCSC Part (none) -> C2906982; Manufacturer (none) -> FOJAN; Manufacturer Part (none) -> FRC0603F1002TS; Unit Price (none) -> 0.001
- renumbered C2 to C5, C3 to C6, D2 to D1, U9 to JR1, U10 to JR2, R22 to R6, SW3 to SW2, SW4 to SW3, SW5 to SW4
Connections:
- net +5V: now also JR1.1 (VCC), JR1.4 (VCC), JR2.1 (VCC), JR2.4 (VCC), R7.1, C1.2, C2.2; no longer JR1.H3 (H+), JR1.V3 (V+), JR2.H3 (H+), JR2.V3 (V+), R7.2
- net CE: now also U1.11 (PCINT23/AIN1/PD7); no longer U1.10 (PCINT22/OC0A/AIN0/PD6)
- net CSN: now also U1.10 (PCINT22/OC0A/AIN0/PD6); no longer U1.11 (PCINT23/AIN1/PD7)
- net GND: now also D1.1 (K), JR1.10 (SW2), JR1.3 (GND), JR1.6 (GND), JR1.8 (SW2), JR2.10 (SW2), JR2.3 (GND), JR2.6 (GND), JR2.8 (SW2), SW3.4, SW4.4, C1.1, C2.1; no longer JR1.B1A (SEL-), JR1.H1 (H-), JR1.V1 (V-), JR2.B1A (SEL-), JR2.H1 (H-), JR2.V1 (V-), R6.1
- net JOY1-B: now also JR1.7 (SW1), JR1.9 (SW1), R7.2; no longer JR1.B2A (SEL+), R7.1
- net JOY1-X: now also JR1.5 (VR2), U1.27 (PC4/ADC4/SDA/PCINT12); no longer JR1.H2 (H), U1.23 (PC0/ADC0/PCINT8)
- net JOY1-Y: now also JR1.2 (VR1), U1.28 (PC5/ADC5/SCL/PCINT13); no longer JR1.V2 (V), U1.24 (PC1/ADC1/PCINT9)
- net JOY2-B: now also JR2.7 (SW1), JR2.9 (SW1), U1.25 (PC2/ADC2/PCINT10); no longer JR2.B2A (SEL+), U1.28 (PC5/ADC5/SCL/PCINT13)
- net JOY2-X: now also JR2.2 (VR1), U1.22 (ADC7); no longer JR2.H2 (H), U1.19 (ADC6)
- net JOY2-Y: now also JR2.5 (VR2), U1.19 (ADC6); no longer JR2.V2 (V), U1.22 (ADC7)
- net MOSI: now also J1.3; no longer J1.1
- net SCK: now also J1.1; no longer J1.3
- net LED: now reaches R6.2
- net LED: now also U1.9 (PCINT21/OC0B/T1/PD5); no longer D1.1 (K)
- net at D1.2 (A): now also R6.1; no longer U1.9 (PCINT21/OC0B/T1/PD5)
- net BTN1: now reaches R5.1, SW3.1
- net BTN1: now also SW3.2, U1.23 (PC0/ADC0/PCINT8); no longer U1.2 (PCINT20/XCK/T0/PD4)
- net BTN2: now reaches R4.1, SW4.1
- net BTN2: now also SW4.2, U1.24 (PC1/ADC1/PCINT9); no longer U1.1 (PCINT19/OC2B/INT1/PD3)
- net at RV1.2: now also U1.26 (PC3/ADC3/PCINT11); no longer U1.27 (PC4/ADC4/SDA/PCINT12)
- new net TOGGLE1: R2.1, SW2.3, U1.1 (PCINT19/OC2B/INT1/PD3)
- new net TOGGLE2: R3.1, SW2.1, U1.2 (PCINT20/XCK/T0/PD4)
- no-connect marks 5 -> 1
Other:
- removed sheet Transceiver
- sheet Display ports: added CS, DC, MOSI, RESET, SCK; removed TFT_CS, TFT_DC, TFT_MISO, TFT_MOSI, TFT_RESET, TFT_SCK
- company: (none) -> 42 Paris
- title: (none) -> Controller
- moved on the sheet: D1, J3, R4, R5, R6, R7, R8, SW2

Commit message: add controller gerber file
Parts:
- removed C3: 100nF, common:C_0603, symbol common:Capacitor
Connections:
- net GND: now also SW1.1
Changed lines of the file:
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@@
 	(wire
 		(pts
-			(xy 36.83 39.37) (xy 26.67 39.37)
+			(xy 26.67 39.37) (xy 46.99 39.37)
 		)
 		(stroke
@@
 	(wire
 		(pts
-			(xy 41.91 39.37) (xy 46.99 39.37)
-		)
-		(stroke
-			(width 0)
-			(type default)
-		)
-	)
-	(wire
-		(pts
 			(xy 153.67 95.25) (xy 165.1 95.25)
 		)
@@
 					(unit 1)
 				)
-			)
-		)
-	)
-	(symbol
-		(lib_id "common:Capacitor")
-		(at 39.37 39.37 0)
-		(unit 1)
-		(exclude_from_sim no)
-		(in_bom yes)
-		(on_board yes)
-		(dnp no)
-		(fields_autoplaced yes)
-		(property "Reference" "C3"
-			(at 39.37 33.02 0)
-			(effects
-				(font
-					(size 1.27 1.27)
-				)
-			)
-		)
-		(property "Value" "100nF"
-			(at 39.37 35.56 0)
-			(effects
-				(font
-					(size 1.27 1.27)
-				)
-			)
-		)
-		(property "Footprint" "common:C_0603"
-			(at 39.37 39.37 0)
-			(effects
-				(font
-					(size 1.27 1.27)
-				)
-				(hide yes)
-			)
-		)
-		(property "Datasheet" ""
-			(at 39.37 39.37 0)
-			(effects
-				(font
-					(size 1.27 1.27)
-				)
-				(hide yes)
-			)
-		)
-		(property "Description" "Unpolarized Capacitor"
-			(at 39.37 44.87 0)
-			(effects
-				(font
-					(size 1.27 1.27)
-				)
-				(hide yes)
-			)
-		)
-		(property "Ext. Price" "0.25"
-			(at 39.37 39.37 0)
-			(effects
-				(font
-					(size 1.27 1.27)
-				)
-				(hide yes)
-			)
-		)
-		(property "LCSC Part" "C14663"
-			(at 39.37 39.37 0)
-			(effects
-				(font
-					(size 1.27 1.27)
-				)
-				(hide yes)
-			)
-		)
-		(property "Manufacturer" "YAGEO"
-			(at 39.37 39.37 0)
-			(effects
-				(font
-					(size 1.27 1.27)
-				)
-				(hide yes)
-			)
-		)
-		(property "Manufacturer Part" "CC0603KRX7R9BB104"
-			(at 39.37 39.37 0)
-			(effects
-				(font
-					(size 1.27 1.27)
-				)
-				(hide yes)
-			)
-		)
-		(property "Unit Price" "0.0025"
-			(at 39.37 39.37 0)
-			(effects
-				(font
-					(size 1.27 1.27)
-				)
-				(hide yes)
-			)
-		)
-		(pin "1"
-		)
-		(pin "2"
-		)
-		(instances
-			(project ""
-				(path "/beaf00ba-d60c-407c-adfe-9d518bae0b16"
-					(reference "C3")
-					(unit 1)
-				)
