File: hardware/boards/vehicles/car/transceiver.kicad_sch (KiCad schematic)
At the start: 31 parts, among them J6 SMA, J7 02x04, U7 NRF24L01, U8 RFX2401C, Y3 16MHz

Commit message: updated main points of the car schematic
Parts:
- C25, C26, C27, C28, C29, C30, C31, C32, C33, C34, C35, C36, C37, C38, C39, C40, J6, L10, L6, L7, L8, L9, R24, R26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: now left out of the parts list
